Commit message: worked on labels for arena wire harness

File: resources/geometries/Clip1/Clip1.urdf (robot description, URDF)
Before this commit: robot Clips_2.SLDPRT, 1 links, 0 joints
Links:
- removed link Clips_2.SLDPRT
- added link Clips_1.SLDPRT, mass 0.0014073; collision mesh filename=package://Clip1/meshes/Clips_1.SLDPRT.STL; visual mesh filename=package://Clip1/meshes/Clips_1.SLDPRT.STL

File: resources/geometries/Clip1_modified/Clip1_modified.urdf (robot description, URDF)
Before this commit: robot Clips_3_modified.SLDPRT, 1 links, 0 joints
Links:
- removed link Clips_3_modified.SLDPRT
- added link Clips_1_modified.SLDPRT, mass 0.0058626; collision mesh filename=package://Clip1_modified/meshes/Clips_1_modified.SLDPRT.STL; visual mesh filename=package://Clip1_modified/meshes/Clips_1_modified.SLDPRT.STL

File: resources/geometries/Clip2/Clip2.urdf (robot description, URDF)
Before this commit: robot Clips_1.SLDPRT, 1 links, 0 joints
Links:
- removed link Clips_1.SLDPRT
- added link Clips_2.SLDPRT, mass 0.00082038; collision mesh filename=package://Clip2/meshes/Clips_2.SLDPRT.STL; visual mesh filename=package://Clip2/meshes/Clips_2.SLDPRT.STL

File: resources/geometries/Clip2_modified/Clip2_modified.urdf (robot description, URDF)
Before this commit: robot Clips_3.SLDPRT, 1 links, 0 joints
Links:
- removed link Clips_3.SLDPRT
- added link Clips_2_modified.SLDPRT, mass 0.0053058; collision mesh filename=package://Clip2_modified/meshes/Clips_2_modified.SLDPRT.STL; visual mesh filename=package://Clip2_modified/meshes/Clips_2_modified.SLDPRT.STL

File: resources/geometries/Clip3/Clip3.urdf (robot description, URDF)
Before this commit: robot Clips_4.SLDPRT, 1 links, 0 joints
Links:
- removed link Clips_4.SLDPRT
- added link Clip3, mass 0.001788; collision mesh filename=package://Clip3/meshes/Clips_3.SLDPRT.STL; visual mesh filename=package://Clip3/meshes/Clips_3.SLDPRT.STL

File: resources/geometries/Clip3_modified/Clip3_modified.urdf (robot description, URDF)
Before this commit: robot Clips_4_modified.SLDPRT, 1 links, 0 joints
Links:
- removed link Clips_4_modified.SLDPRT
- added link Clip3_modified, mass 0.0063855; collision mesh filename=package://Clip3_modified/meshes/Clips_3_modified.SLDPRT.STL; visual mesh filename=package://Clip3_modified/meshes/Clips_3_modified.SLDPRT.STL

File: resources/geometries/Clip4/Clip4.urdf (robot description, URDF)
Before this commit: robot Clips_2_modified.SLDPRT, 1 links, 0 joints
Links:
- removed link Clips_2_modified.SLDPRT
- added link Clips_4.SLDPRT, mass 0.0019621; collision mesh filename=package://Clip4.SLDPRT/meshes/Clips_4.SLDPRT.STL; visual mesh filename=package://Clip4/meshes/Clips_4.SLDPRT.STL

File: resources/geometries/Clip4_modified/Clip4_modified.urdf (robot description, URDF)
Before this commit: robot Clips_1_modified.SLDPRT, 1 links, 0 joints
Links:
- removed link Clips_1_modified.SLDPRT
- added link Clips_4_modified.SLDPRT, mass 0.0065162; collision mesh filename=package://Clip4_modified/meshes/Clips_4_modified.SLDPRT.STL; visual mesh filename=package://Clip4_modified/meshes/Clips_4_modified.SLDPRT.STL
